File: print.kicad_pcb (KiCad board)
At the start: 2 copper layers, 81.3 x 55.9 mm, 74 parts, among them P1 433MHzRx, P2 433MHzTx, P3 B6B-PH-K-S, P4 Conn_01x06, Q1 BC817K-40_215, Q2 BC817K-40_215, Q3 BC817K-40_215, Q4 BC817K-40_215, U1 DS18B20_, U2 SN74LVC1G32DBVR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

Commit message: 2. Marts 2021
Parts:
- P1, P2, P4, RST1, debug1: moved to B.Cu
- VR1: footprint Package_TO_SOT_THT:TO-220-3_Vertical -> Package_TO_SOT_THT:TO-220-3_Horizontal_TabDown
- moved C7 82.5 mm to (134.6, 49.8)
- moved C2 81.8 mm to (131.3, 78.5), turned to 90 degrees
- moved C4 80.7 mm to (137.2, 55.9), turned to 180 degrees
- moved C1 64.7 mm to (106.0, 56.0), turned to -90 degrees
- moved VR1 64.1 mm to (125.5, 49.7)
- moved C5 52.0 mm to (103.6, 93.2), turned to -90 degrees
- moved C3 50.0 mm to (118.4, 49.8), turned to 180 degrees
- moved P1 46.6 mm to (120.4, 69.3)
- moved U2 42.4 mm to (123.3, 73.5), turned to -90 degrees
- moved P2 40.7 mm to (117.1, 69.3)
- moved C6 39.4 mm to (99.1, 87.1), turned to 180 degrees
- moved U3 30.1 mm to (141.3, 51.0)
- moved R8 23.9 mm to (145.8, 50.0), turned to 0 degrees
- moved Heater1 23.3 mm to (145.1, 56.0), turned to 90 degrees
- moved R27 20.7 mm to (145.8, 52.3), turned to 0 degrees
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Connections:
- Module1 pad 17: Net-(Module1-Pad17) -> unconnected-(Module1-Pad17)
- Module1 pad 18: Net-(Module1-Pad18) -> unconnected-(Module1-Pad18)
- Module1 pad 19: Net-(Module1-Pad19) -> unconnected-(Module1-Pad19)
- Module1 pad 20: Net-(Module1-Pad20) -> unconnected-(Module1-Pad20)
- Module1 pad 21: Net-(Module1-Pad21) -> unconnected-(Module1-Pad21)
- Module1 pad 22: Net-(Module1-Pad22) -> unconnected-(Module1-Pad22)
- Module1 pad 32: Net-(Module1-Pad32) -> unconnected-(Module1-Pad32)
- Module2 pad 10: Net-(Module2-Pad10) -> unconnected-(Module2-Pad10)
- Module2 pad 11: Net-(Module2-Pad11) -> unconnected-(Module2-Pad11)
- Module2 pad 15: Net-(Module2-Pad15) -> unconnected-(Module2-Pad15)
- Module2 pad 16: Net-(Module2-Pad16) -> unconnected-(Module2-Pad16)
- Module2 pad 17: Net-(Module2-Pad17) -> unconnected-(Module2-Pad17)
- Module2 pad 18: Net-(Module2-Pad18) -> unconnected-(Module2-Pad18)
- Module2 pad 19: Net-(Module2-Pad19) -> unconnected-(Module2-Pad19)
- Module2 pad 20: Net-(Module2-Pad20) -> unconnected-(Module2-Pad20)
- Module2 pad 23: Net-(Module2-Pad23) -> unconnected-(Module2-Pad23)
- Module2 pad 24: Net-(Module2-Pad24) -> unconnected-(Module2-Pad24)
- Module2 pad 25: Net-(Module2-Pad25) -> unconnected-(Module2-Pad25)
- Module2 pad 26: Net-(Module2-Pad26) -> unconnected-(Module2-Pad26)
- Module2 pad 27: Net-(Module2-Pad27) -> unconnected-(Module2-Pad27)
- Module2 pad 28: Net-(Module2-Pad28) -> unconnected-(Module2-Pad28)
- Module2 pad 29: Net-(Module2-Pad29) -> unconnected-(Module2-Pad29)
- Module2 pad 3: Net-(Module2-Pad3) -> unconnected-(Module2-Pad3)
- Module2 pad 30: Net-(Module2-Pad30) -> unconnected-(Module2-Pad30)
- Module2 pad 33: Net-(Module2-Pad33) -> unconnected-(Module2-Pad33)
- Module2 pad 4: Net-(Module2-Pad4) -> unconnected-(Module2-Pad4)
- Module2 pad 5: Net-(Module2-Pad5) -> unconnected-(Module2-Pad5)
- Module2 pad 6: Net-(Module2-Pad6) -> unconnected-(Module2-Pad6)
- Module2 pad 7: Net-(Module2-Pad7) -> unconnected-(Module2-Pad7)
- Module2 pad 8: Net-(Module2-Pad8) -> unconnected-(Module2-Pad8)
- Module2 pad 9: Net-(Module2-Pad9) -> unconnected-(Module2-Pad9)
- P2 pad 1: Net-(P2-Pad1) -> unconnected-(P2-Pad1)
- U4A1 pad 1: Net-(U4A1-Pad1) -> unconnected-(U4A1-Pad1)
- U4A1 pad 10: Earth -> unconnected-(U4A1-Pad10)
- U4A1 pad 11: Earth -> unconnected-(U4A1-Pad11)
- U4A1 pad 12: Earth -> unconnected-(U4A1-Pad12)
- U4A1 pad 3: Net-(U4A1-Pad3) -> unconnected-(U4A1-Pad3)
- U4A1 pad 4: Net-(U4A1-Pad4) -> unconnected-(U4A1-Pad4)
- U4A1 pad 5: Earth -> unconnected-(U4A1-Pad5)
- U4A1 pad 6: Earth -> unconnected-(U4A1-Pad6)
- U4A1 pad 7: Earth -> unconnected-(U4A1-Pad7)
- U4A1 pad 8: Earth -> unconnected-(U4A1-Pad8)
- U4A1 pad 9: Earth -> unconnected-(U4A1-Pad9)
- debug1 pad 2: Net-(debug1-Pad2) -> unconnected-(debug1-Pad2)
- debug1 pad 3: Net-(debug1-Pad3) -> unconnected-(debug1-Pad3)
- debug1 pad 6: Net-(debug1-Pad6) -> unconnected-(debug1-Pad6)
Other:
- net class Default removed
